File: left/matrix.kicad_sch (KiCad schematic)
At the start: 34 parts

Commit message: removed warnings
Parts:
- KEY1, KEY10, KEY11, KEY12, KEY13, KEY14, KEY15, KEY16, KEY17, KEY2, KEY3, KEY4, KEY5, KEY6, KEY7, KEY8, KEY9: footprint Low Profile Keyswitches:SW_Kailh_Choc_V1_HotSwap_18mm_caps -> Low Profile Keyswitches:SW_Kailh_Choc_V1_HotSwap
Changed lines of the file:
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@@
 			)
 		)
-		(property "Footprint" "Low Profile Keyswitches:SW_Kailh_Choc_V1_HotSwap_18mm_caps"
+		(property "Footprint" "Low Profile Keyswitches:SW_Kailh_Choc_V1_HotSwap"
 			(at 87.63 110.49 0)
 			(hide yes)
@@
 			)
 		)
-		(property "Footprint" "Low Profile Keyswitches:SW_Kailh_Choc_V1_HotSwap_18mm_caps"
+		(property "Footprint" "Low Profile Keyswitches:SW_Kailh_Choc_V1_HotSwap"
 			(at 182.88 110.49 0)
 			(hide yes)
@@
 			)
 		)
-		(property "Footprint" "Low Profile Keyswitches:SW_Kailh_Choc_V1_HotSwap_18mm_caps"
+		(property "Footprint" "Low Profile Keyswitches:SW_Kailh_Choc_V1_HotSwap"
 			(at 87.63 87.63 0)
 			(hide yes)
@@
 			)
 		)
-		(property "Footprint" "Low Profile Keyswitches:SW_Kailh_Choc_V1_HotSwap_18mm_caps"
+		(property "Footprint" "Low Profile Keyswitches:SW_Kailh_Choc_V1_HotSwap"
 			(at 151.13 110.49 0)
 			(hide yes)
@@
 			)
 		)
-		(property "Footprint" "Low Profile Keyswitches:SW_Kailh_Choc_V1_HotSwap_18mm_caps"
+		(property "Footprint" "Low Profile Keyswitches:SW_Kailh_Choc_V1_HotSwap"
 			(at 119.38 110.49 0)
 			(hide yes)
@@
 			)
 		)
-		(property "Footprint" "Low Profile Keyswitches:SW_Kailh_Choc_V1_HotSwap_18mm_caps"
+		(property "Footprint" "Low Profile Keyswitches:SW_Kailh_Choc_V1_HotSwap"
 			(at 151.13 64.77 0)
 			(hide yes)
@@
 			)
 		)
-		(property "Footprint" "Low Profile Keyswitches:SW_Kailh_Choc_V1_HotSwap_18mm_caps"
+		(property "Footprint" "Low Profile Keyswitches:SW_Kailh_Choc_V1_HotSwap"
 			(at 214.63 87.63 0)
 			(hide yes)
@@
 			)
 		)
-		(property "Footprint" "Low Profile Keyswitches:SW_Kailh_Choc_V1_HotSwap_18mm_caps"
+		(property "Footprint" "Low Profile Keyswitches:SW_Kailh_Choc_V1_HotSwap"
 			(at 182.88 133.35 0)
 			(hide yes)
@@
 			)
 		)
-		(property "Footprint" "Low Profile Keyswitches:SW_Kailh_Choc_V1_HotSwap_18mm_caps"
+		(property "Footprint" "Low Profile Keyswitches:SW_Kailh_Choc_V1_HotSwap"
 			(at 151.13 87.63 0)
 			(hide yes)
@@
 			)
 		)
-		(property "Footprint" "Low Profile Keyswitches:SW_Kailh_Choc_V1_HotSwap_18mm_caps"
+		(property "Footprint" "Low Profile Keyswitches:SW_Kailh_Choc_V1_HotSwap"
 			(at 87.63 64.77 0)
 			(hide yes)
@@
 			)
 		)
-		(property "Footprint" "Low Profile Keyswitches:SW_Kailh_Choc_V1_HotSwap_18mm_caps"
+		(property "Footprint" "Low Profile Keyswitches:SW_Kailh_Choc_V1_HotSwap"
 			(at 182.88 87.63 0)
 			(hide yes)
@@
 			)
 		)
-		(property "Footprint" "Low Profile Keyswitches:SW_Kailh_Choc_V1_HotSwap_18mm_caps"
+		(property "Footprint" "Low Profile Keyswitches:SW_Kailh_Choc_V1_HotSwap"
 			(at 214.63 133.35 0)
 			(hide yes)
@@
 			)
 		)
-		(property "Footprint" "Low Profile Keyswitches:SW_Kailh_Choc_V1_HotSwap_18mm_caps"
+		(property "Footprint" "Low Profile Keyswitches:SW_Kailh_Choc_V1_HotSwap"
 			(at 214.63 64.77 0)
 			(hide yes)
@@
 			)
 		)
-		(property "Footprint" "Low Profile Keyswitches:SW_Kailh_Choc_V1_HotSwap_18mm_caps"
+		(property "Footprint" "Low Profile Keyswitches:SW_Kailh_Choc_V1_HotSwap"
 			(at 214.63 110.49 0)
 			(hide yes)
@@
 			)
 		)
-		(property "Footprint" "Low Profile Keyswitches:SW_Kailh_Choc_V1_HotSwap_18mm_caps"
+		(property "Footprint" "Low Profile Keyswitches:SW_Kailh_Choc_V1_HotSwap"
 			(at 119.38 87.63 0)
 			(hide yes)
@@
 			)
 		)
-		(property "Footprint" "Low Profile Keyswitches:SW_Kailh_Choc_V1_HotSwap_18mm_caps"
+		(property "Footprint" "Low Profile Keyswitches:SW_Kailh_Choc_V1_HotSwap"
 			(at 182.88 64.77 0)
 			(hide yes)
@@
 			)
 		)
-		(property "Footprint" "Low Profile Keyswitches:SW_Kailh_Choc_V1_HotSwap_18mm_caps"
+		(property "Footprint" "Low Profile Keyswitches:SW_Kailh_Choc_V1_HotSwap"
 			(at 119.38 64.77 0)
 			(hide yes)

Commit message: redesigned pcb
Parts:
- KEY1, KEY10, KEY11, KEY12, KEY13, KEY14, KEY15, KEY16, KEY17, KEY2, KEY3, KEY4, KEY5, KEY6, KEY7, KEY8, KEY9: footprint Low Profile Keyswitches:SW_Kailh_Choc_V1_HotSwap -> Low Profile Keyswitches:SW_Kailh_Choc_V1_HotSwap_18mm_caps
Changed lines of the file:
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@@
 			)
 		)
-		(property "Footprint" "Low Profile Keyswitches:SW_Kailh_Choc_V1_HotSwap"
+		(property "Footprint" "Low Profile Keyswitches:SW_Kailh_Choc_V1_HotSwap_18mm_caps"
 			(at 87.63 110.49 0)
 			(hide yes)
@@
 			)
 		)
-		(property "Footprint" "Low Profile Keyswitches:SW_Kailh_Choc_V1_HotSwap"
+		(property "Footprint" "Low Profile Keyswitches:SW_Kailh_Choc_V1_HotSwap_18mm_caps"
 			(at 182.88 110.49 0)
 			(hide yes)
@@
 			)
 		)
-		(property "Footprint" "Low Profile Keyswitches:SW_Kailh_Choc_V1_HotSwap"
+		(property "Footprint" "Low Profile Keyswitches:SW_Kailh_Choc_V1_HotSwap_18mm_caps"
 			(at 87.63 87.63 0)
 			(hide yes)
@@
 			)
 		)
-		(property "Footprint" "Low Profile Keyswitches:SW_Kailh_Choc_V1_HotSwap"
+		(property "Footprint" "Low Profile Keyswitches:SW_Kailh_Choc_V1_HotSwap_18mm_caps"
 			(at 151.13 110.49 0)
 			(hide yes)
@@
 			)
 		)
-		(property "Footprint" "Low Profile Keyswitches:SW_Kailh_Choc_V1_HotSwap"
+		(property "Footprint" "Low Profile Keyswitches:SW_Kailh_Choc_V1_HotSwap_18mm_caps"
 			(at 119.38 110.49 0)
 			(hide yes)
@@
 			)
 		)
-		(property "Footprint" "Low Profile Keyswitches:SW_Kailh_Choc_V1_HotSwap"
+		(property "Footprint" "Low Profile Keyswitches:SW_Kailh_Choc_V1_HotSwap_18mm_caps"
 			(at 151.13 64.77 0)
 			(hide yes)
@@
 			)
 		)
-		(property "Footprint" "Low Profile Keyswitches:SW_Kailh_Choc_V1_HotSwap"
+		(property "Footprint" "Low Profile Keyswitches:SW_Kailh_Choc_V1_HotSwap_18mm_caps"
 			(at 214.63 87.63 0)
 			(hide yes)
@@
 			)
 		)
-		(property "Footprint" "Low Profile Keyswitches:SW_Kailh_Choc_V1_HotSwap"
+		(property "Footprint" "Low Profile Keyswitches:SW_Kailh_Choc_V1_HotSwap_18mm_caps"
 			(at 182.88 133.35 0)
 			(hide yes)
@@
 			)
 		)
-		(property "Footprint" "Low Profile Keyswitches:SW_Kailh_Choc_V1_HotSwap"
+		(property "Footprint" "Low Profile Keyswitches:SW_Kailh_Choc_V1_HotSwap_18mm_caps"
 			(at 151.13 87.63 0)
 			(hide yes)
@@
 			)
 		)
-		(property "Footprint" "Low Profile Keyswitches:SW_Kailh_Choc_V1_HotSwap"
+		(property "Footprint" "Low Profile Keyswitches:SW_Kailh_Choc_V1_HotSwap_18mm_caps"
 			(at 87.63 64.77 0)
 			(hide yes)
@@
 			)
 		)
-		(property "Footprint" "Low Profile Keyswitches:SW_Kailh_Choc_V1_HotSwap"
+		(property "Footprint" "Low Profile Keyswitches:SW_Kailh_Choc_V1_HotSwap_18mm_caps"
 			(at 182.88 87.63 0)
 			(hide yes)
@@
 			)
 		)
-		(property "Footprint" "Low Profile Keyswitches:SW_Kailh_Choc_V1_HotSwap"
+		(property "Footprint" "Low Profile Keyswitches:SW_Kailh_Choc_V1_HotSwap_18mm_caps"
 			(at 214.63 133.35 0)
 			(hide yes)
@@
 			)
 		)
-		(property "Footprint" "Low Profile Keyswitches:SW_Kailh_Choc_V1_HotSwap"
+		(property "Footprint" "Low Profile Keyswitches:SW_Kailh_Choc_V1_HotSwap_18mm_caps"
 			(at 214.63 64.77 0)
 			(hide yes)
@@
 			)
 		)
-		(property "Footprint" "Low Profile Keyswitches:SW_Kailh_Choc_V1_HotSwap"
+		(property "Footprint" "Low Profile Keyswitches:SW_Kailh_Choc_V1_HotSwap_18mm_caps"
 			(at 214.63 110.49 0)
 			(hide yes)
@@
 			)
 		)
-		(property "Footprint" "Low Profile Keyswitches:SW_Kailh_Choc_V1_HotSwap"
+		(property "Footprint" "Low Profile Keyswitches:SW_Kailh_Choc_V1_HotSwap_18mm_caps"
 			(at 119.38 87.63 0)
 			(hide yes)
@@
 			)
 		)
-		(property "Footprint" "Low Profile Keyswitches:SW_Kailh_Choc_V1_HotSwap"
+		(property "Footprint" "Low Profile Keyswitches:SW_Kailh_Choc_V1_HotSwap_18mm_caps"
 			(at 182.88 64.77 0)
 			(hide yes)
@@
 			)
 		)
-		(property "Footprint" "Low Profile Keyswitches:SW_Kailh_Choc_V1_HotSwap"
+		(property "Footprint" "Low Profile Keyswitches:SW_Kailh_Choc_V1_HotSwap_18mm_caps"
 			(at 119.38 64.77 0)
 			(hide yes)
