File: left/left.kicad_pcb (KiCad board)
At the start: 2 copper layers, 117.6 x 97.9 mm, 53 parts, among them J1 USB_C_Receptacle_IN, J2 USB_C_Receptacle_OUT, SW1 SW_Push, SW2 SW_SPDT, U1 STM32G0B1CBTx, U2 SRV05-4, U3 XC6206P332MR, U4 SRV05-4

Commit message: sent to jcl for production
Parts:
- R1, SW1, SW2: moved to F.Cu
- moved R1 1.01 mm to (82.0, 111.2)
- turned SW2 to 0 degrees
Connections:
- U2 pad 1: TX -> unconnected-(U2-IO1-Pad1)
- U2 pad 6: RX -> unconnected-(U2-IO4-Pad6)
Routing:
- net TX: track 59.3 -> 55.6 mm
- net RX: track 56.5 -> 54.6 mm
- net GND: track 19.2 -> 17.4 mm
- net nRST: track 38.4 -> 40.0 mm, vias 2 -> 3
- net +3.3V: track 147.7 -> 148.8 mm, vias 4 -> 3
- net BOOT0: track 6.94 -> 6.00 mm, vias 0 -> 1
Other:
- board text added: "Flashing"
- board text added: "Normal"
- board text added: "{dblquote}What's that black thing?{dblquote}"
