File: left/left.kicad_pcb (KiCad board)
At the start: 2 copper layers, 117.6 x 97.9 mm, 53 parts, among them J1 USB_C_Receptacle_IN, J2 USB_C_Receptacle_OUT, SW1 SW_Push, SW2 SW_SPDT, U1 STM32G0B1CBTx, U2 SRV05-4, U3 XC6206P332MR, U4 SRV05-4

Commit message: compiled new files for production
Parts:
- KEY1, KEY10, KEY11, KEY12, KEY13, KEY14, KEY15, KEY16, KEY17, KEY2, KEY3, KEY4, KEY5, KEY6, KEY7, KEY8, KEY9: footprint Keyswitch Marbastlib Choc:SW_choc_v1_HS_CPG135001S30_1u -> marbastlib-choc:SW_choc_v1_HS_CPG135001S30_1u

Commit message: added new production files for left side
Routing:
- net GND: vias 37 -> 38
Other:
- outline, holes or cut-outs redrawn
Changed lines of the file:
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@@
 		(tags "capacitor handsolder")
 		(property "Reference" "C3"
-			(at 2.74375 -0.01875 90)
+			(at -2.67 -0.01875 90)
 			(layer "B.SilkS")
 			(effects
@@
 		)
 		(pad "2" smd roundrect
-			(at -3.245 -5.949998 170)
+			(at -3.245 -5.949997 170)
 			(size 2.65 2.6)
 			(layers "B.Cu" "B.Mask" "B.Paste")
@@
 		(tags "capacitor handsolder")
 		(property "Reference" "C2"
-			(at 2.74375 0 90)
+			(at -2.67 0.01 90)
 			(layer "B.SilkS")
 			(effects
@@
 		(tags "capacitor handsolder")
 		(property "Reference" "C4"
-			(at 2.74375 0.03125 90)
+			(at -2.67 0.03125 90)
 			(layer "B.SilkS")
 			(effects
@@
 		(tags "capacitor handsolder")
 		(property "Reference" "C1"
-			(at 2.74375 -0.00625 90)
+			(at -2.67 -0.00625 90)
 			(layer "B.SilkS")
 			(effects
@@
 	)
 	(gr_circle
-		(center 115.2 119.7)
-		(end 113.2 119.7)
+		(center 117.43 109.65)
+		(end 115.43 109.65)
 		(stroke
 			(width 0.05)
@@
 		(size 0.6)
 		(drill 0.3)
+		(layers "F.Cu" "B.Cu")
+		(free yes)
+		(net "GND")
+	)
+	(via
+		(at 98.5 107.8)
+		(size 0.6)
+		(drill 0.3)

Commit message: pushed usb a bit outwards for better fitting with the case
Parts:
- moved J2 0.70 mm to (146.0, 112.1)
- moved J1 0.68 mm to (49.8, 66.9)
Routing:
- net +5V: track 226.2 -> 229.3 mm
- net D-: track 80.7 -> 82.9 mm
- net D+: track 85.8 -> 88.0 mm
- net RX: track 53.8 -> 55.9 mm
- net Net-(J1-CC2): track 5.66 -> 6.77 mm
- net Net-(J1-CC1): track 6.65 -> 7.76 mm
- net TX: track 56.1 -> 56.8 mm
- net VBUS: track 16.1 -> 15.6 mm
Other:
- outline, holes or cut-outs redrawn
