File: right/matrix.kicad_sch (KiCad schematic)
At the start: 34 parts

Commit message: unverified done right
Parts:
- KEY1, KEY10, KEY11, KEY12, KEY13, KEY14, KEY15, KEY16, KEY17, KEY2, KEY3, KEY4, KEY5, KEY6, KEY7, KEY8, KEY9: footprint Low Profile Keyswitches:SW_Kailh_Choc_V1_HotSwap_18mm_caps -> Low Profile Keyswitches:SW_Kailh_Choc_V1_HotSwap
Changed lines of the file:
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@@
 			)
 		)
-		(property "Footprint" "Low Profile Keyswitches:SW_Kailh_Choc_V1_HotSwap_18mm_caps"
+		(property "Footprint" "Low Profile Keyswitches:SW_Kailh_Choc_V1_HotSwap"
 			(at 124.46 93.98 0)
 			(hide yes)
@@
 			)
 		)
-		(property "Footprint" "Low Profile Keyswitches:SW_Kailh_Choc_V1_HotSwap_18mm_caps"
+		(property "Footprint" "Low Profile Keyswitches:SW_Kailh_Choc_V1_HotSwap"
 			(at 219.71 116.84 0)
 			(hide yes)
@@
 			)
 		)
-		(property "Footprint" "Low Profile Keyswitches:SW_Kailh_Choc_V1_HotSwap_18mm_caps"
+		(property "Footprint" "Low Profile Keyswitches:SW_Kailh_Choc_V1_HotSwap"
 			(at 92.71 71.12 0)
 			(hide yes)
@@
 			)
 		)
-		(property "Footprint" "Low Profile Keyswitches:SW_Kailh_Choc_V1_HotSwap_18mm_caps"
+		(property "Footprint" "Low Profile Keyswitches:SW_Kailh_Choc_V1_HotSwap"
 			(at 156.21 71.12 0)
 			(hide yes)
@@
 			)
 		)
-		(property "Footprint" "Low Profile Keyswitches:SW_Kailh_Choc_V1_HotSwap_18mm_caps"
+		(property "Footprint" "Low Profile Keyswitches:SW_Kailh_Choc_V1_HotSwap"
 			(at 156.21 116.84 0)
 			(hide yes)
@@
 			)
 		)
-		(property "Footprint" "Low Profile Keyswitches:SW_Kailh_Choc_V1_HotSwap_18mm_caps"
+		(property "Footprint" "Low Profile Keyswitches:SW_Kailh_Choc_V1_HotSwap"
 			(at 187.96 116.84 0)
 			(hide yes)
@@
 			)
 		)
-		(property "Footprint" "Low Profile Keyswitches:SW_Kailh_Choc_V1_HotSwap_18mm_caps"
+		(property "Footprint" "Low Profile Keyswitches:SW_Kailh_Choc_V1_HotSwap"
 			(at 124.46 116.84 0)
 			(hide yes)
@@
 			)
 		)
-		(property "Footprint" "Low Profile Keyswitches:SW_Kailh_Choc_V1_HotSwap_18mm_caps"
+		(property "Footprint" "Low Profile Keyswitches:SW_Kailh_Choc_V1_HotSwap"
 			(at 124.46 71.12 0)
 			(hide yes)
@@
 			)
 		)
-		(property "Footprint" "Low Profile Keyswitches:SW_Kailh_Choc_V1_HotSwap_18mm_caps"
+		(property "Footprint" "Low Profile Keyswitches:SW_Kailh_Choc_V1_HotSwap"
 			(at 219.71 93.98 0)
 			(hide yes)
@@
 			)
 		)
-		(property "Footprint" "Low Profile Keyswitches:SW_Kailh_Choc_V1_HotSwap_18mm_caps"
+		(property "Footprint" "Low Profile Keyswitches:SW_Kailh_Choc_V1_HotSwap"
 			(at 92.71 116.84 0)
 			(hide yes)
@@
 			)
 		)
-		(property "Footprint" "Low Profile Keyswitches:SW_Kailh_Choc_V1_HotSwap_18mm_caps"
+		(property "Footprint" "Low Profile Keyswitches:SW_Kailh_Choc_V1_HotSwap"
 			(at 92.71 93.98 0)
 			(hide yes)
@@
 			)
 		)
-		(property "Footprint" "Low Profile Keyswitches:SW_Kailh_Choc_V1_HotSwap_18mm_caps"
+		(property "Footprint" "Low Profile Keyswitches:SW_Kailh_Choc_V1_HotSwap"
 			(at 156.21 93.98 0)
 			(hide yes)
@@
 			)
 		)
-		(property "Footprint" "Low Profile Keyswitches:SW_Kailh_Choc_V1_HotSwap_18mm_caps"
+		(property "Footprint" "Low Profile Keyswitches:SW_Kailh_Choc_V1_HotSwap"
 			(at 187.96 71.12 0)
 			(hide yes)
@@
 			)
 		)
-		(property "Footprint" "Low Profile Keyswitches:SW_Kailh_Choc_V1_HotSwap_18mm_caps"
+		(property "Footprint" "Low Profile Keyswitches:SW_Kailh_Choc_V1_HotSwap"
 			(at 187.96 93.98 0)
 			(hide yes)
@@
 			)
 		)
-		(property "Footprint" "Low Profile Keyswitches:SW_Kailh_Choc_V1_HotSwap_18mm_caps"
+		(property "Footprint" "Low Profile Keyswitches:SW_Kailh_Choc_V1_HotSwap"
 			(at 92.71 139.7 0)
 			(hide yes)
@@
 			)
 		)
-		(property "Footprint" "Low Profile Keyswitches:SW_Kailh_Choc_V1_HotSwap_18mm_caps"
+		(property "Footprint" "Low Profile Keyswitches:SW_Kailh_Choc_V1_HotSwap"
 			(at 124.46 139.7 0)
 			(hide yes)
@@
 			)
 		)
-		(property "Footprint" "Low Profile Keyswitches:SW_Kailh_Choc_V1_HotSwap_18mm_caps"
+		(property "Footprint" "Low Profile Keyswitches:SW_Kailh_Choc_V1_HotSwap"
 			(at 219.71 71.12 0)
 			(hide yes)

Commit message: fixed schematics
Parts:
- KEY1, KEY10, KEY11, KEY12, KEY13, KEY14, KEY15, KEY16, KEY17, KEY2, KEY3, KEY4, KEY5, KEY6, KEY7, KEY8, KEY9: footprint Low Profile Keyswitches:SW_Kailh_Choc_V1_HotSwap -> Keyswitches Marbastlib Choc:SW_choc_v1_HS_CPG135001S30_1u
Changed lines of the file:
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@@
 			)
 		)
-		(property "Footprint" "Low Profile Keyswitches:SW_Kailh_Choc_V1_HotSwap"
+		(property "Footprint" "Keyswitches Marbastlib Choc:SW_choc_v1_HS_CPG135001S30_1u"
 			(at 124.46 93.98 0)
 			(hide yes)
@@
 			)
 		)
-		(property "Footprint" "Low Profile Keyswitches:SW_Kailh_Choc_V1_HotSwap"
+		(property "Footprint" "Keyswitches Marbastlib Choc:SW_choc_v1_HS_CPG135001S30_1u"
 			(at 219.71 116.84 0)
 			(hide yes)
@@
 			)
 		)
-		(property "Footprint" "Low Profile Keyswitches:SW_Kailh_Choc_V1_HotSwap"
+		(property "Footprint" "Keyswitches Marbastlib Choc:SW_choc_v1_HS_CPG135001S30_1u"
 			(at 92.71 71.12 0)
 			(hide yes)
@@
 			)
 		)
-		(property "Footprint" "Low Profile Keyswitches:SW_Kailh_Choc_V1_HotSwap"
+		(property "Footprint" "Keyswitches Marbastlib Choc:SW_choc_v1_HS_CPG135001S30_1u"
 			(at 156.21 71.12 0)
 			(hide yes)
@@
 			)
 		)
-		(property "Footprint" "Low Profile Keyswitches:SW_Kailh_Choc_V1_HotSwap"
+		(property "Footprint" "Keyswitches Marbastlib Choc:SW_choc_v1_HS_CPG135001S30_1u"
 			(at 156.21 116.84 0)
 			(hide yes)
@@
 			)
 		)
-		(property "Footprint" "Low Profile Keyswitches:SW_Kailh_Choc_V1_HotSwap"
+		(property "Footprint" "Keyswitches Marbastlib Choc:SW_choc_v1_HS_CPG135001S30_1u"
 			(at 187.96 116.84 0)
 			(hide yes)
@@
 			)
 		)
-		(property "Footprint" "Low Profile Keyswitches:SW_Kailh_Choc_V1_HotSwap"
+		(property "Footprint" "Keyswitches Marbastlib Choc:SW_choc_v1_HS_CPG135001S30_1u"
 			(at 124.46 116.84 0)
 			(hide yes)
@@
 			)
 		)
-		(property "Footprint" "Low Profile Keyswitches:SW_Kailh_Choc_V1_HotSwap"
+		(property "Footprint" "Keyswitches Marbastlib Choc:SW_choc_v1_HS_CPG135001S30_1u"
 			(at 124.46 71.12 0)
 			(hide yes)
@@
 			)
 		)
-		(property "Footprint" "Low Profile Keyswitches:SW_Kailh_Choc_V1_HotSwap"
+		(property "Footprint" "Keyswitches Marbastlib Choc:SW_choc_v1_HS_CPG135001S30_1u"
 			(at 219.71 93.98 0)
 			(hide yes)
@@
 			)
 		)
-		(property "Footprint" "Low Profile Keyswitches:SW_Kailh_Choc_V1_HotSwap"
+		(property "Footprint" "Keyswitches Marbastlib Choc:SW_choc_v1_HS_CPG135001S30_1u"
 			(at 92.71 116.84 0)
 			(hide yes)
@@
 			)
 		)
-		(property "Footprint" "Low Profile Keyswitches:SW_Kailh_Choc_V1_HotSwap"
+		(property "Footprint" "Keyswitches Marbastlib Choc:SW_choc_v1_HS_CPG135001S30_1u"
 			(at 92.71 93.98 0)
 			(hide yes)
@@
 			)
 		)
-		(property "Footprint" "Low Profile Keyswitches:SW_Kailh_Choc_V1_HotSwap"
+		(property "Footprint" "Keyswitches Marbastlib Choc:SW_choc_v1_HS_CPG135001S30_1u"
 			(at 156.21 93.98 0)
 			(hide yes)
@@
 			)
 		)
-		(property "Footprint" "Low Profile Keyswitches:SW_Kailh_Choc_V1_HotSwap"
+		(property "Footprint" "Keyswitches Marbastlib Choc:SW_choc_v1_HS_CPG135001S30_1u"
 			(at 187.96 71.12 0)
 			(hide yes)
@@
 			)
 		)
-		(property "Footprint" "Low Profile Keyswitches:SW_Kailh_Choc_V1_HotSwap"
+		(property "Footprint" "Keyswitches Marbastlib Choc:SW_choc_v1_HS_CPG135001S30_1u"
 			(at 187.96 93.98 0)
 			(hide yes)
@@
 			)
 		)
-		(property "Footprint" "Low Profile Keyswitches:SW_Kailh_Choc_V1_HotSwap"
+		(property "Footprint" "Keyswitches Marbastlib Choc:SW_choc_v1_HS_CPG135001S30_1u"
 			(at 92.71 139.7 0)
 			(hide yes)
@@
 			)
 		)
-		(property "Footprint" "Low Profile Keyswitches:SW_Kailh_Choc_V1_HotSwap"
+		(property "Footprint" "Keyswitches Marbastlib Choc:SW_choc_v1_HS_CPG135001S30_1u"
 			(at 124.46 139.7 0)
 			(hide yes)
@@
 			)
 		)
-		(property "Footprint" "Low Profile Keyswitches:SW_Kailh_Choc_V1_HotSwap"
+		(property "Footprint" "Keyswitches Marbastlib Choc:SW_choc_v1_HS_CPG135001S30_1u"
 			(at 219.71 71.12 0)
 			(hide yes)

Commit message: v3 for the right side
Parts:
- KEY1, KEY10, KEY11, KEY12, KEY13, KEY14, KEY15, KEY16, KEY17, KEY2, KEY3, KEY4, KEY5, KEY6, KEY7, KEY8, KEY9: footprint Keyswitches Marbastlib Choc:SW_choc_v1_HS_CPG135001S30_1u -> Keyswitches Marbastlib:SW_choc_v1_HS_CPG135001S30_1u
Changed lines of the file:
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@@
 			)
 		)
-		(property "Footprint" "Keyswitches Marbastlib Choc:SW_choc_v1_HS_CPG135001S30_1u"
+		(property "Footprint" "Keyswitches Marbastlib:SW_choc_v1_HS_CPG135001S30_1u"
 			(at 124.46 93.98 0)
 			(hide yes)
@@
 			)
 		)
-		(property "Footprint" "Keyswitches Marbastlib Choc:SW_choc_v1_HS_CPG135001S30_1u"
+		(property "Footprint" "Keyswitches Marbastlib:SW_choc_v1_HS_CPG135001S30_1u"
 			(at 219.71 116.84 0)
 			(hide yes)
@@
 			)
 		)
-		(property "Footprint" "Keyswitches Marbastlib Choc:SW_choc_v1_HS_CPG135001S30_1u"
+		(property "Footprint" "Keyswitches Marbastlib:SW_choc_v1_HS_CPG135001S30_1u"
 			(at 92.71 71.12 0)
 			(hide yes)
@@
 			)
 		)
-		(property "Footprint" "Keyswitches Marbastlib Choc:SW_choc_v1_HS_CPG135001S30_1u"
+		(property "Footprint" "Keyswitches Marbastlib:SW_choc_v1_HS_CPG135001S30_1u"
 			(at 156.21 71.12 0)
 			(hide yes)
@@
 			)
 		)
-		(property "Footprint" "Keyswitches Marbastlib Choc:SW_choc_v1_HS_CPG135001S30_1u"
+		(property "Footprint" "Keyswitches Marbastlib:SW_choc_v1_HS_CPG135001S30_1u"
 			(at 156.21 116.84 0)
 			(hide yes)
@@
 			)
 		)
-		(property "Footprint" "Keyswitches Marbastlib Choc:SW_choc_v1_HS_CPG135001S30_1u"
+		(property "Footprint" "Keyswitches Marbastlib:SW_choc_v1_HS_CPG135001S30_1u"
 			(at 187.96 116.84 0)
 			(hide yes)
@@
 			)
 		)
-		(property "Footprint" "Keyswitches Marbastlib Choc:SW_choc_v1_HS_CPG135001S30_1u"
+		(property "Footprint" "Keyswitches Marbastlib:SW_choc_v1_HS_CPG135001S30_1u"
 			(at 124.46 116.84 0)
 			(hide yes)
@@
 			)
 		)
-		(property "Footprint" "Keyswitches Marbastlib Choc:SW_choc_v1_HS_CPG135001S30_1u"
+		(property "Footprint" "Keyswitches Marbastlib:SW_choc_v1_HS_CPG135001S30_1u"
 			(at 124.46 71.12 0)
 			(hide yes)
@@
 			)
 		)
-		(property "Footprint" "Keyswitches Marbastlib Choc:SW_choc_v1_HS_CPG135001S30_1u"
+		(property "Footprint" "Keyswitches Marbastlib:SW_choc_v1_HS_CPG135001S30_1u"
 			(at 219.71 93.98 0)
 			(hide yes)
@@
 			)
 		)
-		(property "Footprint" "Keyswitches Marbastlib Choc:SW_choc_v1_HS_CPG135001S30_1u"
+		(property "Footprint" "Keyswitches Marbastlib:SW_choc_v1_HS_CPG135001S30_1u"
 			(at 92.71 116.84 0)
 			(hide yes)
@@
 			)
 		)
-		(property "Footprint" "Keyswitches Marbastlib Choc:SW_choc_v1_HS_CPG135001S30_1u"
+		(property "Footprint" "Keyswitches Marbastlib:SW_choc_v1_HS_CPG135001S30_1u"
 			(at 92.71 93.98 0)
 			(hide yes)
@@
 			)
 		)
-		(property "Footprint" "Keyswitches Marbastlib Choc:SW_choc_v1_HS_CPG135001S30_1u"
+		(property "Footprint" "Keyswitches Marbastlib:SW_choc_v1_HS_CPG135001S30_1u"
 			(at 156.21 93.98 0)
 			(hide yes)
@@
 			)
 		)
-		(property "Footprint" "Keyswitches Marbastlib Choc:SW_choc_v1_HS_CPG135001S30_1u"
+		(property "Footprint" "Keyswitches Marbastlib:SW_choc_v1_HS_CPG135001S30_1u"
 			(at 187.96 71.12 0)
 			(hide yes)
@@
 			)
 		)
-		(property "Footprint" "Keyswitches Marbastlib Choc:SW_choc_v1_HS_CPG135001S30_1u"
+		(property "Footprint" "Keyswitches Marbastlib:SW_choc_v1_HS_CPG135001S30_1u"
 			(at 187.96 93.98 0)
 			(hide yes)
@@
 			)
 		)
-		(property "Footprint" "Keyswitches Marbastlib Choc:SW_choc_v1_HS_CPG135001S30_1u"
+		(property "Footprint" "Keyswitches Marbastlib:SW_choc_v1_HS_CPG135001S30_1u"
 			(at 92.71 139.7 0)
 			(hide yes)
@@
 			)
 		)
-		(property "Footprint" "Keyswitches Marbastlib Choc:SW_choc_v1_HS_CPG135001S30_1u"
+		(property "Footprint" "Keyswitches Marbastlib:SW_choc_v1_HS_CPG135001S30_1u"
 			(at 124.46 139.7 0)
 			(hide yes)
@@
 			)
 		)
-		(property "Footprint" "Keyswitches Marbastlib Choc:SW_choc_v1_HS_CPG135001S30_1u"
+		(property "Footprint" "Keyswitches Marbastlib:SW_choc_v1_HS_CPG135001S30_1u"
 			(at 219.71 71.12 0)
 			(hide yes)
